File: hw/shiftregister-tester.sch (KiCad schematic (older format))
At the start: 2 parts, among them U1 74LS165

Commit message: two LEDs to show status
Parts:
- added D1, D2: LED, symbol Device:LED
- added R1, R2: 1k, symbol Device:R
- TB1: symbol ARDUINO_NANO:ARDUINO_NANO -> shiftregister-tester-rescue:ARDUINO_NANO-ARDUINO_NANO
- U1: symbol 74xx:74LS165 -> shiftregister-tester-rescue:74LS165-74xx
Connections:
- net GND: now also D1.1 (K), D2.1 (K)
- net at TB1.13 (D10): now also R1.2
- net at TB1.14 (D11/MOSI): now also R2.2
- new net: D1.2 (A), R1.1
- new net: D2.2 (A), R2.1
Changed lines of the file:
@@
 $EndDescr
 $Comp
-L ARDUINO_NANO:ARDUINO_NANO TB1
+L shiftregister-tester-rescue:ARDUINO_NANO-ARDUINO_NANO TB1
 U 1 1 5D66DDCB
 P 4200 3600
@@
 $EndComp
 $Comp
-L power:+5V #PWR?
+L power:+5V #PWR0101
 U 1 1 5D66DEB9
 P 5050 2300
-F 0 "#PWR?" H 5050 2150 50  0001 C CNN
+F 0 "#PWR0101" H 5050 2150 50  0001 C CNN
 F 1 "+5V" H 5065 2473 50  0000 C CNN
 F 2 "" H 5050 2300 50  0001 C CNN
@@
 $EndComp
 $Comp
-L power:GND #PWR?
+L power:GND #PWR0102
 U 1 1 5D66DEF8
 P 5050 2500
-F 0 "#PWR?" H 5050 2250 50  0001 C CNN
+F 0 "#PWR0102" H 5050 2250 50  0001 C CNN
 F 1 "GND" H 5055 2327 50  0000 C CNN
 F 2 "" H 5050 2500 50  0001 C CNN
@@
 $EndComp
 $Comp
-L 74xx:74LS165 U1
+L shiftregister-tester-rescue:74LS165-74xx U1
 U 1 1 5D66DF54
 P 6850 2850
@@
 $EndComp
 $Comp
-L power:+5V #PWR?
+L power:+5V #PWR0103
 U 1 1 5D66E004
 P 7150 1950
-F 0 "#PWR?" H 7150 1800 50  0001 C CNN
+F 0 "#PWR0103" H 7150 1800 50  0001 C CNN
 F 1 "+5V" H 7165 2123 50  0000 C CNN
 F 2 "" H 7150 1950 50  0001 C CNN
@@
 $EndComp
 $Comp
-L power:GND #PWR?
+L power:GND #PWR0104
 U 1 1 5D66E035
 P 6850 4000
-F 0 "#PWR?" H 6850 3750 50  0001 C CNN
+F 0 "#PWR0104" H 6850 3750 50  0001 C CNN
 F 1 "GND" H 6855 3827 50  0000 C CNN
 F 2 "" H 6850 4000 50  0001 C CNN
@@
 Wire Wire Line
 	6850 3900 6850 4000
+$Comp
+L Device:R R1
+U 1 1 5D6B1799
+P 5550 4450
+F 0 "R1" H 5480 4404 50  0000 R CNN
+F 1 "1k" H 5480 4495 50  0000 R CNN
+F 2 "" V 5480 4450 50  0001 C CNN
+F 3 "~" H 5550 4450 50  0001 C CNN
+	1    5550 4450
+	-1   0    0    1
+$EndComp
+$Comp
+L Device:R R2
+U 1 1 5D6B17F1
+P 5200 4450
+F 0 "R2" H 5130 4404 50  0000 R CNN
+F 1 "1k" H 5130 4495 50  0000 R CNN
+F 2 "" V 5130 4450 50  0001 C CNN
+F 3 "~" H 5200 4450 50  0001 C CNN
+	1    5200 4450
+	-1   0    0    1
+$EndComp
+Wire Wire Line
+	4900 4300 5200 4300
+Wire Wire Line
+	4900 4200 5550 4200
+Wire Wire Line
+	5550 4200 5550 4300
+$Comp
+L Device:LED D2
+U 1 1 5D6B1F1F
+P 5200 4750
+F 0 "D2" V 5238 4633 50  0000 R CNN
+F 1 "LED" V 5147 4633 50  0000 R CNN
+F 2 "" H 5200 4750 50  0001 C CNN
+F 3 "~" H 5200 4750 50  0001 C CNN
+	1    5200 4750
+	0    -1   -1   0
+$EndComp
+$Comp
+L Device:LED D1
+U 1 1 5D6B1F92
+P 5550 4750
+F 0 "D1" V 5588 4633 50  0000 R CNN
+F 1 "LED" V 5497 4633 50  0000 R CNN
+F 2 "" H 5550 4750 50  0001 C CNN
+F 3 "~" H 5550 4750 50  0001 C CNN
+	1    5550 4750
+	0    -1   -1   0
+$EndComp
+Wire Wire Line
+	5200 5000 5550 5000
+Wire Wire Line
+	5550 5000 5550 4900
+Wire Wire Line
+	5550 5000 5550 5050
+Connection ~ 5550 5000
+$Comp
+L power:GND #PWR0105
+U 1 1 5D6B21A9
+P 5550 5050
+F 0 "#PWR0105" H 5550 4800 50  0001 C CNN
+F 1 "GND" H 5555 4877 50  0000 C CNN
+F 2 "" H 5550 5050 50  0001 C CNN
+F 3 "" H 5550 5050 50  0001 C CNN
+	1    5550 5050
+	1    0    0    -1
+$EndComp
+Wire Wire Line
+	5200 4900 5200 5000
 $EndSCHEMATC

Commit message: RDIN goes from the shift register to the Arduino
Parts:
- TB1: symbol shiftregister-tester-rescue:ARDUINO_NANO-ARDUINO_NANO -> shiftregister-tester-rescue:ARDUINO_NANO-ARDUINO_NANO-shiftregister-tester-rescue
- U1: symbol shiftregister-tester-rescue:74LS165-74xx -> shiftregister-tester-rescue:74LS165-74xx-shiftregister-tester-rescue
Connections:
- no-connect marks 1 -> 2
Changed lines of the file:
@@
 $EndDescr
 $Comp
-L shiftregister-tester-rescue:ARDUINO_NANO-ARDUINO_NANO TB1
+L shiftregister-tester-rescue:ARDUINO_NANO-ARDUINO_NANO-shiftregister-tester-rescue TB1
 U 1 1 5D66DDCB
 P 4200 3600
@@
 $EndComp
 $Comp
-L shiftregister-tester-rescue:74LS165-74xx U1
+L shiftregister-tester-rescue:74LS165-74xx-shiftregister-tester-rescue U1
 U 1 1 5D66DF54
 P 6850 2850
@@
 Text GLabel 4900 4100 2    50   Input ~ 0
 D7
-Text GLabel 3500 3000 0    50   Output ~ 0
+Text GLabel 3500 3000 0    50   Input ~ 0
 RDIN
-Text GLabel 7350 2250 2    50   Input ~ 0
+Text GLabel 7350 2250 2    50   Output ~ 0
 RDIN
 Text GLabel 3500 3100 0    50   Output ~ 0
@@
 Wire Wire Line
 	5200 4900 5200 5000
+NoConn ~ 3500 3400
 $EndSCHEMATC
